File: pcb/main.sch (EAGLE design)
At the start: 5 parts

Commit message: change i2c line
Parts:
- removed HTU2X: (no value), pinhead:PINHD-1X4
- removed JP_DISPLAY: (no value), pinhead:PINHD-1X5
- removed PH1: BPX81, opto-trans-siemens:BPX81
- added BAT, SERVICE: (no value), pinhead:PINHD-1X2
- added I2C, I2C1: (no value), pinhead:PINHD-1X4
- added R2: 10k, resistor:R-EU_R0805
Connections:
- removed net +3V3: HTU2X.1, R1.2, U$2.3V3
- removed net N$11: JP_DISPLAY.5, U$2.4
- removed net N$5: HTU2X.4, U$2.9
- removed net N$6: JP_DISPLAY.4, U$2.5
- new net N$3: I2C.4, I2C1.4, U$2.7
- net +5V: now also BAT.1, I2C.1, I2C1.1, R1.2, U$2.3V3; no longer JP_DISPLAY.1, U$2.5V
- net GND: now also BAT.2, I2C.2, I2C1.2, R2.1, SERVICE.2; no longer HTU2X.2, JP_DISPLAY.2, PH1.E
- net N$1: now also I2C.3, I2C1.3; no longer JP_DISPLAY.3
- net N$2: now also R2.2; no longer PH1.C
- net N$4: now also SERVICE.1, U$2.1; no longer HTU2X.3, U$2.8
